File: pcb/Keychain-tris.kicad_pcb (KiCad board)
At the start: 2 copper layers, 41 x 33 mm, 40 parts, among them J1 Conn_01x02, J2 USB_C_Receptacle_USB2.0_16P, J3 Conn_01x04, J4 Conn_01x08, J5 Conn_01x08, SW1 TS24CA, SW2 TS24CA, U1 ESP32-C3, U2 AMS1117-3.3, U3 MPU-6050_C24112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

Commit message: fixes
Routing:
- net GND: vias 17 -> 19
Other:
- board size 41 x 33 mm -> 40.7 x 33.6 mm
- board text added: "Keychain-Tris!!"
Changed lines of the file:
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@@
 		(embedded_fonts no)
 		(model "${KICAD9_3DMODEL_DIR}/Connector_PinSocket_2.54mm.3dshapes/PinSocket_1x02_P2.54mm_Vertical.wrl"
+			(hide yes)
 			(offset
 				(xyz 0 0 0)
@@
 			)
 		)
+		(model "${KIPRJMOD}/lib/USB-C_SMD-TYPE-C-31-M-12_1.step"
+			(offset
+				(xyz 0 -1 0)
+			)
+			(scale
+				(xyz 1 1 1)
+			)
+			(rotate
+				(xyz -0 -0 -180)
+			)
+		)
 	)
 	(footprint "Capacitor_SMD:C_0805_2012Metric"
@@
 		)
 		(embedded_fonts no)
-		(model "${KICAD9_3DMODEL_DIR}/Connector_PinSocket_2.54mm.3dshapes/PinSocket_1x08_P2.54mm_Vertical.wrl"
-			(offset
-				(xyz 0 0 0)
-			)
-			(scale
-				(xyz 1 1 1)
-			)
-			(rotate
-				(xyz 0 0 0)
-			)
-		)
 	)
 	(footprint "Package_DFN_QFN:QFN-32-1EP_5x5mm_P0.5mm_EP3.7x3.7mm"
@@
 		)
 		(embedded_fonts no)
-		(model "${KICAD9_3DMODEL_DIR}/Connector_PinSocket_2.54mm.3dshapes/PinSocket_1x08_P2.54mm_Vertical.wrl"
-			(offset
-				(xyz 0 0 0)
-			)
-			(scale
-				(xyz 1 1 1)
-			)
-			(rotate
-				(xyz 0 0 0)
-			)
-		)
 	)
 	(footprint "Capacitor_SMD:C_0805_2012Metric"
@@
 	)
 	(gr_line
-		(start 116.9 42.2)
-		(end 116.9 47.3)
+		(start 121.6 72)
+		(end 114.2 72)
 		(stroke
 			(width 0.05)
@@
 	)
 	(gr_line
-		(start 130.1 60.8)
-		(end 130.1 74.2)
+		(start 124.7 46.9)
+		(end 124.7 53.3)
 		(stroke
 			(width 0.05)
@@
 	)
 	(gr_line
-		(start 121.5 74.2)
-		(end 121.5 72.1)
+		(start 121.6 74.2)
+		(end 121.6 72)
 		(stroke
 			(width 0.05)
@@
 	)
 	(gr_line
-		(start 129.4 60.8)
-		(end 130.1 60.8)
+		(start 98.1 75.4)
+		(end 98.1 74.1)
 		(stroke
 			(width 0.05)
@@
 		(layer "Edge.Cuts")
 	)
-	(gr_line
-		(start 121.5 72.1)
-		(end 114 72.1)
+	(gr_circle
+		(center 91.8 44.82132)
+		(end 93.3 46.32132)
 		(stroke
 			(width 0.05)
 			(type default)
 		)
+		(fill no)
 		(layer "Edge.Cuts")
 	)
 	(gr_line
-		(start 129.4 74.2)
-		(end 121.5 74.2)
+		(start 129.8 62.4)
+		(end 129.8 74.2)
 		(stroke
 			(width 0.05)
@@
 	)
 	(gr_line
-		(start 89.1 60.7)
-		(end 92.4 60.7)
+		(start 114.2 72)
+		(end 114.2 75.4)
 		(stroke
 			(width 0.05)
@@
 	)
 	(gr_line
-		(start 97.4 75.1)
-		(end 97.4 73.3)
+		(start 127 60.6)
+		(end 129.8 60.6)
 		(stroke
 			(width 0.05)
@@
 	)
 	(gr_line
-		(start 114 72.1)
-		(end 114 75.1)
+		(start 117.4 41.8)
+		(end 117.4 46.9)
 		(stroke
 			(width 0.05)
@@
 	)
 	(gr_line
-		(start 97.4 73.3)
-		(end 89.1 73.3)
+		(start 129.8 74.2)
+		(end 121.6 74.2)
 		(stroke
 			(width 0.05)
@@
 	)
 	(gr_line
-		(start 114 75.2)
-		(end 97.4 75.2)
+		(start 117.4 46.9)
+		(end 124.7 46.9)
 		(stroke
 			(width 0.05)
@@
 	)
 	(gr_line
-		(start 114 75.2)
-		(end 114 75.1)
+		(start 89.1 41.95)
+		(end 89.1 41.8)
 		(stroke
 			(width 0.05)
@@
 	)
 	(gr_line
-		(start 124.2 53.9)
-		(end 126.5 53.9)
+		(start 89.1 74.1)
+		(end 89.1 41.95)
 		(stroke
 			(width 0.05)
@@
 	)
 	(gr_line
-		(start 124.2 47.3)
-		(end 124.2 53.9)
+		(start 114.2 75.4)
+		(end 98.1 75.4)
 		(stroke
 			(width 0.05)
@@
 	)
 	(gr_line
-		(start 126.5 53.9)
-		(end 126.5 60.8)
+		(start 98.1 74.1)
+		(end 89.1 74.1)
 		(stroke
 			(width 0.05)
@@
 	)
 	(gr_line
-		(start 92.4 42.2)
-		(end 116.9 42.2)
+		(start 92.2 41.8)
+		(end 89.1 41.8)
 		(stroke
 			(width 0.05)
@@
 	)
 	(gr_line
-		(start 129.4 74.2)
-		(end 130.1 74.2)
+		(start 127 53.3)
+		(end 127 60.6)
 		(stroke
 			(width 0.05)
@@
 	)
 	(gr_line
-		(start 126.5 60.8)
-		(end 129.4 60.8)
+		(start 124.7 53.3)
+		(end 127 53.3)
 		(stroke
 			(width 0.05)
@@
 	)
 	(gr_line
-		(start 116.9 47.3)
-		(end 124.2 47.3)
+		(start 92.2 41.8)
+		(end 117.4 41.8)
 		(stroke
 			(width 0.05)
@@
 	)
 	(gr_line
-		(start 89.1 73.3)
-		(end 89.1 60.7)
+		(start 129.8 60.6)
+		(end 129.8 62.4)
 		(stroke
 			(width 0.05)
@@
 		(layer "Edge.Cuts")
 	)
-	(gr_line
-		(start 92.4 60.7)
-		(end 92.4 42.2)
-		(stroke
-			(width 0.05)
-			(type default)
+	(gr_text "Keychain-Tris!!"
+		(at 91.6 60.5 90)
+		(layer "F.SilkS")
+		(effects
+			(font
+				(size 1 1)
+				(thickness 0.1)
+			)
+			(justify left bottom)
 		)
-		(layer "Edge.Cuts")
 	)
 	(segment
@@
 	)
 	(via
+		(at 116.2 65.4)
+		(size 0.6)
+		(drill 0.3)
+		(layers "F.Cu" "B.Cu")
+		(net 1)
+	)
+	(via
 		(at 94.7 55.6)
 		(size 0.6)
@@
 		(size 0.6)
 		(drill 0.3)
+		(layers "F.Cu" "B.Cu")
+		(net 1)
+	)
+	(via
+		(at 114.4 69.8)
+		(size 0.6)
+		(drill 0.3)
